Commit message: diff

File: backend/engine/data/humanoid/humanoid.urdf (robot description, URDF)
Before this commit: robot dumpUrdf, 16 links, 15 joints
Links:
- link left_ankle: geometry collision box size=0.26 0.34 0.06; collision box size=0.708000 0.220000 0.360000
- link right_ankle: geometry collision box size=0.26 0.34 0.06; collision box size=0.708000 0.220000 0.360000

Commit message: diff

File: backend/engine/data/humanoid/humanoid.urdf (robot description, URDF)
Before this commit: robot dumpUrdf, 16 links, 15 joints
Links:
- link left_ankle: geometry collision box size=0.34 0.06 0.26; collision box size=0.708000 0.220000 0.360000
- link right_ankle: geometry collision box size=0.34 0.06 0.26; collision box size=0.708000 0.220000 0.360000

Commit message: spinal

File: backend/engine/data/humanoid/humanoid.urdf (robot description, URDF)
Before this commit: robot dumpUrdf, 16 links, 15 joints
Links:
- added link spine, mass 4.000000; collision sphere radius=0.300000
Joints:
- added joint spine: type spherical, parent root, child spine, origin xyz=0.000000 0.472302 0.000000 rpy=0 0 0, axis 0 0 1
- joint chest: origin xyz=0.000000 0.944604 0.000000 rpy=0 0 0 -> xyz=0.000000 0.472302 0.000000 rpy=0 0 0; parent root -> spine

Commit message: diff

File: backend/engine/data/humanoid/humanoid.urdf (robot description, URDF)
Before this commit: robot dumpUrdf, 17 links, 16 joints
Links:
- link left_ankle: geometry collision box size=0.44 0.08 0.30; collision box size=0.780000 0.300000 0.400000
- link right_ankle: geometry collision box size=0.44 0.08 0.30; collision box size=0.780000 0.300000 0.400000
Joints:
- joint left_hip: origin xyz=0.000000 0.000000 -0.339548 rpy=0 0 0 -> xyz=0.000000 0.000000 -0.425000 rpy=0 0 0
- joint right_hip: origin xyz=0.000000 0.000000 0.339548 rpy=0 0 0 -> xyz=0.000000 0.000000 0.425000 rpy=0 0 0

Commit message: Fix backward falling and learning: larger feet, forward lean, intervention loss
Physics stability:
- URDF feet: main box 0.78→1.10, sole 0.44→0.70, shifted forward
  (COM of foot moved from 0.18 to 0.22 for better forward support)
- Foot mass: 1.0→1.2 for better ground contact
- Spine pitch bias: 0.50→0.54 (slight forward lean like humans)

Causal learning (critical fix):
- l_int was ALWAYS 0 despite LAMBDA_INT=2.0 being defined. The
  intervention prediction loss was never applied. Now properly
  computes extra MSE loss on intervention batch with 4x weight
- LAMBDA_L1: 0.02→0.005 (was pruning edges faster than they formed)
- LAMBDA_INT: 2.0→4.0 (stronger intervention signal)
- LAMBDA_DAG: 0.5→0.3 (less aggressive DAG constraint)
- EDGE_THRESH: 0.05→0.04 (retain weaker discovered edges)
- Default passive_mix: 0.35→0.15 (less passive, more causal data)

Co-authored-by: Andrew Yefymenko <Andruefim@users.noreply.github.com>

File: backend/engine/data/humanoid/humanoid.urdf (robot description, URDF)
Before this commit: robot dumpUrdf, 17 links, 16 joints
Links:
- link left_ankle: mass 1.000000 -> 1.200000; geometry collision box size=0.70 0.10 0.44; collision box size=1.100000 0.300000 0.500000
- link right_ankle: mass 1.000000 -> 1.200000; geometry collision box size=0.70 0.10 0.44; collision box size=1.100000 0.300000 0.500000

Commit message: Update humanoid URDF masses and inertias for 35kg robot at globalScaling=0.225
Set URDF masses so that world_mass = urdf_mass × 0.225³ produces
Unitree G1-proportioned body segments totaling 35 kg.
Inertia values scaled proportionally (~62× increase).

Co-authored-by: Andrew Yefymenko <Andruefim@users.noreply.github.com>

File: backend/engine/data/humanoid/humanoid.urdf (robot description, URDF)
Before this commit: robot dumpUrdf, 17 links, 16 joints
Links:
- link chest: mass 14.000000 -> 870.8
- link left_ankle: mass 1.200000 -> 74.6
- link left_elbow: mass 1.000000 -> 62.0
- link left_hip: mass 4.500000 -> 280.0
- link left_knee: mass 3.000000 -> 187.0
- link left_shoulder: mass 1.500000 -> 93.0
- link left_wrist: mass 0.500000 -> 31.0
- link neck: mass 2.000000 -> 124.4
- link right_ankle: mass 1.200000 -> 74.6
- link right_elbow: mass 1.000000 -> 62.0
- link right_hip: mass 4.500000 -> 280.0
- link right_knee: mass 3.000000 -> 187.0
- link right_shoulder: mass 1.500000 -> 93.0
- link right_wrist: mass 0.500000 -> 31.0
- link root: mass 6.000000 -> 373.0
- link spine: mass 4.000000 -> 248.5

Commit message: Center foot geometry under ankle — fixes backward falling
Root cause: foot collision was offset +0.22 forward (URDF X) from ankle,
placing the support polygon center 5cm ahead of the pelvis/COM.
The COM was behind the support polygon → constant backward falling.

Fix: center foot at (0.0, -0.09, 0.0) instead of (0.22, -0.09, 0.0).
Now support polygon is symmetric around ankle: ±0.11m front/back.
Sole also centered at (0.0, -0.09, -0.14).

Result: pitch stabilizes at -0.003 rad (was -0.09 to -1.5), 0 falls
in 4000 idle steps, 0 falls in 200 interventions.

Co-authored-by: Andrew Yefymenko <Andruefim@users.noreply.github.com>

File: backend/engine/data/humanoid/humanoid.urdf (robot description, URDF)
Before this commit: robot dumpUrdf, 17 links, 16 joints
Links:
- link left_ankle: geometry collision box size=0.80 0.08 0.44; collision box size=1.000000 0.260000 0.500000
- link right_ankle: geometry collision box size=0.80 0.08 0.44; collision box size=1.000000 0.260000 0.500000

Commit message: Fix Г-shape: make chest joint FIXED — was uncontrolled 93° collapse
Root cause: the chest joint (spine→chest, index 2) was a spherical
joint with NO motor control assigned. _apply_motor_intents and set_joint
only control spine_pitch/spine_yaw (joint index 1). The chest joint
had no PD targets, so gravity collapsed it to 93° forward bend.

Fix: change chest joint from 'spherical' to 'fixed'. The spine joint
still provides controlled torso articulation via spine_pitch/spine_yaw.

Result: posture=0.996, pitch=-0.001 rad after 400 agent steps.

Co-authored-by: Andrew Yefymenko <Andruefim@users.noreply.github.com>

File: backend/engine/data/humanoid/humanoid.urdf (robot description, URDF)
Before this commit: robot dumpUrdf, 17 links, 16 joints
Joints:
- joint chest: axis 0 0 1 -> (none); type spherical -> fixed

Commit message: fix weight

File: backend/engine/data/humanoid/humanoid.urdf (robot description, URDF)
Before this commit: robot dumpUrdf, 17 links, 16 joints
Links:
- link chest: mass 870.8 -> 28.0
- link left_ankle: mass 74.6 -> 1.5
- link left_elbow: mass 62.0 -> 2.0
- link left_hip: mass 280.0 -> 9.0
- link left_knee: mass 187.0 -> 4.5
- link left_shoulder: mass 93.0 -> 3.0
- link left_wrist: mass 31.0 -> 0.5
- link neck: mass 124.4 -> 4.0
- link right_ankle: mass 74.6 -> 1.5
- link right_elbow: mass 62.0 -> 2.0
- link right_hip: mass 280.0 -> 9.0
- link right_knee: mass 187.0 -> 4.5
- link right_shoulder: mass 93.0 -> 3.0
- link right_wrist: mass 31.0 -> 0.5
- link root: mass 373.0 -> 12.0
- link spine: mass 248.5 -> 8.0
Joints:
- joint left_wrist: origin xyz=0.000000 -1.035788 0.000000 rpy=0 0 0 -> rpy=0 0.000000 -1.035788 0.000000

Commit message: diff

File: backend/engine/data/humanoid/humanoid.urdf (robot description, URDF)
Before this commit: robot dumpUrdf, 17 links, 16 joints
Links:
- added link head, mass 3.387097; collision sphere radius=0.036923; visual sphere radius=0.036923
- link chest: mass 28.0 -> 21.075269; geometry collision sphere radius=0.135385
- link left_ankle: mass 1.5 -> 1.129032; geometry collision box size=0.246154 0.024615 0.135385; collision box size=0.307692 0.08 0.153846
- link left_elbow: mass 2.0 -> 1.505376; geometry collision capsule length=0.166154 radius=0.049231
- link left_hip: mass 9.0 -> 6.774194; geometry collision capsule length=0.369231 radius=0.067692
- link left_knee: mass 4.5 -> 3.387097; geometry collision capsule length=0.381538 radius=0.061538
- link left_shoulder: mass 3.0 -> 2.258065; geometry collision capsule length=0.221538 radius=0.055385
- link left_wrist: mass 0.5 -> 0.376344; geometry collision sphere radius=0.049231
- link neck: mass 4.0 -> 3.010753; geometry collision sphere radius=0.126154
- link right_ankle: mass 1.5 -> 1.129032; geometry collision box size=0.246154 0.024615 0.135385; collision box size=0.307692 0.08 0.153846
- link right_elbow: mass 2.0 -> 1.505376; geometry collision capsule length=0.166154 radius=0.049231
- link right_hip: mass 9.0 -> 6.774194; geometry collision capsule length=0.369231 radius=0.067692
- link right_knee: mass 4.5 -> 3.387097; geometry collision capsule length=0.381538 radius=0.061538
- link right_shoulder: mass 3.0 -> 2.258065; geometry collision capsule length=0.221538 radius=0.055385
- link right_wrist: mass 0.5 -> 0.376344; geometry collision sphere radius=0.049231
- link root: mass 12.0 -> 9.032258; geometry collision sphere radius=0.110769
- link spine: mass 8.0 -> 6.021505; geometry collision sphere radius=0.092308
Joints:
- added joint head: type fixed, parent neck, child head, origin xyz=0 0.341538 0 rpy=0 0 0
- joint chest: origin xyz=0.000000 0.472302 0.000000 rpy=0 0 0 -> xyz=0 0.145324 0 rpy=0 0 0
- joint left_ankle: origin xyz=0.000000 -1.639480 0.000000 rpy=0 0 0 -> xyz=0 -0.504455 0 rpy=0 0 0
- joint left_elbow: origin xyz=0.000000 -1.099152 0.000000 rpy=0 0 0 -> xyz=0 -0.338201 0 rpy=0 0 0
- joint left_hip: origin xyz=0.000000 0.000000 -0.425000 rpy=0 0 0 -> xyz=0 0 -0.130769 rpy=0 0 0
- joint left_knee: origin xyz=0.000000 -1.686184 0.000000 rpy=0 0 0 -> xyz=0 -0.518826 0 rpy=0 0 0
- joint left_shoulder: origin xyz=-0.096200 0.974000 -0.732440 rpy=0 0 0 -> xyz=-0.0296 0.299692 -0.225366 rpy=0 0 0
- joint left_wrist: axis (none) -> 0 0 1; limit (none) -> lower=-0.8 upper=0.8 effort=200 velocity=2; origin rpy=0 0.000000 -1.035788 0.000000 -> xyz=0 -0.318704 0 rpy=0 0 0; type fixed -> revolute
- joint neck: origin xyz=0.000000 0.895576 0.000000 rpy=0 0 0 -> xyz=0 0.275562 0 rpy=0 0 0
- joint right_ankle: origin xyz=0.000000 -1.639480 0.000000 rpy=0 0 0 -> xyz=0 -0.504455 0 rpy=0 0 0
- joint right_elbow: origin xyz=0.000000 -1.099152 0.000000 rpy=0 0 0 -> xyz=0 -0.338201 0 rpy=0 0 0
- joint right_hip: origin xyz=0.000000 0.000000 0.425000 rpy=0 0 0 -> xyz=0 0 0.130769 rpy=0 0 0
- joint right_knee: origin xyz=0.000000 -1.686184 0.000000 rpy=0 0 0 -> xyz=0 -0.518826 0 rpy=0 0 0
- joint right_shoulder: origin xyz=-0.096200 0.974000 0.732440 rpy=0 0 0 -> xyz=-0.0296 0.299692 0.225366 rpy=0 0 0
- joint right_wrist: axis (none) -> 0 0 1; limit (none) -> lower=-0.8 upper=0.8 effort=200 velocity=2; origin xyz=0.000000 -1.035788 0.000000 rpy=0 0 0 -> xyz=0 -0.318704 0 rpy=0 0 0; type fixed -> revolute
- joint root: origin xyz=0.000000 0.000000 0.000000 rpy=0 0 0 -> xyz=0 0 0 rpy=0 0 0
- joint spine: origin xyz=0.000000 0.472302 0.000000 rpy=0 0 0 -> xyz=0 0.145324 0 rpy=0 0 0

Commit message: diff

File: backend/engine/data/humanoid/humanoid.urdf (robot description, URDF)
Before this commit: robot dumpUrdf, 18 links, 17 joints
Links:
- link neck: mass 3.010753 -> 2.35; geometry collision sphere radius=0.072
Joints:
- joint head: origin xyz=0 0.341538 0 rpy=0 0 0 -> xyz=0 0.202 0 rpy=0 0 0

Commit message: remove wrist

File: backend/engine/data/humanoid/humanoid.urdf (robot description, URDF)
Before this commit: robot dumpUrdf, 18 links, 17 joints
Joints:
- joint left_wrist: axis 0 0 1 -> (none); limit lower=-0.8 upper=0.8 effort=200 velocity=2 -> (none); type revolute -> fixed
- joint right_wrist: axis 0 0 1 -> (none); limit lower=-0.8 upper=0.8 effort=200 velocity=2 -> (none); type revolute -> fixed
